File: goose45.kicad_sch (KiCad schematic)
At the start: 65 parts

Commit message: clean project
* update sch from goose60
Parts:
- removed BOOT?, RST?: DTSM-6, dtsm:KSEM31GLFS, symbol dtsjw:DTSM-6
- removed C?: 1u, 0805:0805C, symbol device:C
- removed C? (x4): 100n, 0805:0805C, symbol device:C
- removed C? (x2): 22p, 0805:0805C, symbol device:C
- removed DF? (x7): LED, symbol device:LED
- removed DF? (x5), DW? (x4): LED, mx1a:MX1A-led_no3d, symbol device:LED
- removed J?: MINI, usb:67503, symbol oupiin_usb:USBMINI_B05
- removed P? (x23): CONN_1, symbol conn:CONN_1
- removed R? (x2): 10k, 0805:0805R, symbol device:R
- removed R? (x10): R, symbol device:R
- removed R? (x2): 22, 0805:0805R, symbol device:R
- removed U?: STM32F103C8Tx, Package_QFP:LQFP-48_7x7mm_P0.5mm, symbol MCU_ST_STM32F1:STM32F103C8Tx
- removed X?: ASX3F, ndk:4-SMD, symbol aker:ASX4
Connections:
- no-connect marks 5 -> 0
Other:
- removed sheet Matrix
- note removed: "Backlight expansion connector (top)"
- note removed: "Universal expansion connector (bottom)"

Commit message: update key switch location on pcb
Parts:
- added C1, C2: 22pF/50V, Capacitor_SMD:C_0603_1608Metric, symbol Device:C_Small
- added C3: 1uF/16V, Capacitor_SMD:C_0603_1608Metric, symbol Device:C_Small
- added C4, C5, C6, C7: 100nF/16V, Capacitor_SMD:C_0603_1608Metric, symbol Device:C_Small
- added D1, D2, D3: LED, LED_SMD:LED_0805_2012Metric, symbol Device:LED
- added H1, H7: MountingHole, MountingHole:MountingHole_3.2mm_M3_Pad, symbol Mechanical:MountingHole
- added H10, H11, H12, H2, H3, H4, H5, H6, H8, H9: MountingHole, MountingHole:MountingHole_3.2mm_M3_Pad_TopOnly, symbol Mechanical:MountingHole
- added R1, R10, R11, R12, R13, R14, R3, R5, R6, R7, R8, R9: 10K/5%, Resistor_SMD:R_0603_1608Metric, symbol Device:R_Small_US
- added R15: 330R/5%, Resistor_SMD:R_0603_1608Metric, symbol Device:R_Small_US
- added R2, R4: 100K/5%, Resistor_SMD:R_0603_1608Metric, symbol Device:R_Small_US
- added SW1, SW2: SW_Push, Button_Switch_SMD:SW_Push_1P1T_NO_CK_KSC6xxJ, symbol Switch:SW_Push
- added U1: STM32F103CBTx, Package_QFP:LQFP-48_7x7mm_P0.5mm, symbol MCU_ST_STM32F1:STM32F103CBTx
- added X1: Crystal_GND24, Crystal:Crystal_SMD_TXC_7M-4Pin_3.2x2.5mm, symbol Device:Crystal_GND24
Connections:
- new net: R4.1, SW2.1
- new net: R1.2, SW1.2
- new net: D1.1 (K), D2.1 (K), D3.1 (K), R15.1
- new net +3.3V: C3.1, C4.1, C5.1, C6.1, C7.1, D1.2 (A), D2.2 (A), D3.2 (A), R1.1, R3.1, R5.1, R7.1, R9.1, U1.1 (VBAT), U1.24 (VDD), U1.36 (VDD), U1.48 (VDD), U1.9 (VDDA)
- new net BOOT0: R2.1, SW1.1, U1.44 (BOOT0)
- new net CAPS_LED: R15.2, U1.29 (PA8)
- new net GND: C1.2, C2.2, C3.2, C4.2, C5.2, C6.2, C7.2, R10.2, R11.1, R12.1, R13.1, R14.1, R2.2, R4.2, R6.2, R8.2, U1.23 (VSS), U1.35 (VSS), U1.47 (VSS), U1.8 (VSSA), X1.2, X1.4
- new net MCU_RX: U1.31 (PA10)
- new net MCU_TX: U1.30 (PA9)
- new net MISO: U1.16 (PA6)
- new net MOSI: U1.17 (PA7)
- new net PA1: R11.2, U1.11 (PA1)
- new net PA3: R12.2, U1.13 (PA3)
- new net PA4: R13.2, U1.14 (PA4)
- new net PB10: R14.2, U1.21 (PB10)
- new net PC13: R10.1, R9.2, U1.2 (PC13)
- new net PC14: R7.2, R8.1, U1.3 (PC14)
- new net PC15: R5.2, R6.1, U1.4 (PC15)
- new net RESET: R3.2, SW2.2, U1.7 (NRST)
- new net SCK: U1.15 (PA5)
- new net SWCLK: U1.37 (PA14)
- new net SWDIO: U1.34 (PA13)
- new net USB_D+: U1.33 (PA12)
- new net USB_D-: U1.32 (PA11)
- new net USB_EN: U1.20 (PB2)
- new net XTAL1: C1.1, U1.5 (PD0), X1.1
- new net XTAL2: C2.1, U1.6 (PD1), X1.3
- new net col1: U1.27 (PB14)
- new net col10: U1.46 (PB9)
- new net col11: U1.18 (PB0)
- new net col12: U1.19 (PB1)
- new net col13: U1.22 (PB11)
- new net col2: U1.26 (PB13)
- new net col3: U1.25 (PB12)
- new net col4: U1.28 (PB15)
- new net col5: U1.39 (PB3)
- new net col6: U1.40 (PB4)
- new net col7: U1.41 (PB5)
- new net col8: U1.42 (PB6)
- new net col9: U1.43 (PB7)
- new net row1: U1.10 (PA0)
- new net row2: U1.45 (PB8)
- new net row3: U1.12 (PA2)
- new net row4: U1.38 (PA15)
Other:
- added sheet Interface (Interface.kicad_sch)
- added sheet PowerManager (PowerManager.kicad_sch)
- added sheet keyswitches (switches.kicad_sch)
