File: goose45rev1/goose45.kicad_pcb (KiCad board)
At the start: 2 copper layers, 247 x 74.8 mm, 145 parts, among them J1 USB_C_Receptacle_USB2.0, J2 SPI, J3 Debugger, J4 USB connector, J5 USART, SW1 Conn_01x02_Female, SW10 SW_Push, SW11 SW_Push, SW12 SW_Push, SW13 SW_Push, SW14 SW_Push, SW15 SW_Push, SW16 SW_Push, SW17 SW_Push, SW18 SW_Push, SW19 SW_Push, SW2 SW_Push, SW20 SW_Push, SW21 SW_Push, SW22 SW_Push, SW23 SW_Push, SW24 SW_Push, SW25 SW_Push, SW26 SW_Push, SW27 SW_Push, SW28 SW_Push, SW29 SW_Push, SW3 SW_Push, SW30 SW_Push, SW31 SW_Push, SW32 SW_Push, SW33 SW_Push, SW34 SW_Push, SW35 SW_Push, SW36 SW_Push, SW37 SW_Push, SW38 SW_Push, SW39 SW_Push, SW39_1 SW_Push, SW4 SW_Push, SW40 SW_Push, SW40_1 SW_Push, SW41 SW_Push, SW41_1 SW_Push, SW42 SW_Push, SW43 SW_Push, SW44 SW_Push, SW44_1 SW_Push, SW45 SW_Push, SW46 SW_Push, SW48 SW_Push, SW5 SW_Push, SW6 SW_Push, SW7 SW_Push, SW8 SW_Push, SW9 SW_Push, U1 STM32F103CBTx, U2 USBLC6-2SC6, U3 TLV75533PDBV, X1 Crystal_GND24

Commit message: change goose45 main board edge.cuts
Parts:
- moved D48 3.19 mm to (270.9, 77.8)
- moved R12 1.36 mm to (30.1, 114.7)
- moved R5 1.36 mm to (30.1, 113.1)
- moved R6 1.36 mm to (30.1, 116.2)
Routing:
- net Net-(D48-Pad2): track 10.2 -> 7.32 mm
- net GND: track 393.9 -> 392.0 mm, vias 313 -> 314
- net PA2: track 27.9 -> 29.0 mm
- net PA4: track 28.4 -> 29.5 mm
- net PA3: track 27.5 -> 28.6 mm
- net row4: track 300.1 -> 301.0 mm
Other:
- outline, holes or cut-outs redrawn

Commit message: update goose45 pcb board edge comment
* goose45 - update board layout
* usbport - change edge size and add edge comment
* usbhub2.0 - change layout and the footprint
Parts:
- moved D38 0.06 mm to (264.2, 113.7)
Routing:
- net row2: track 270.0 -> 265.4 mm
- net row3: track 263.1 -> 259.7 mm
- net row4: track 301.0 -> 297.8 mm
- net VIN: track 68.3 -> 65.0 mm
- net col11: track 243.5 -> 240.8 mm
- net col5: track 163.9 -> 161.4 mm
- net col1: track 89.5 -> 91.3 mm
- net GND: track 392.0 -> 393.8 mm, vias 314 -> 325
- net col9: track 194.6 -> 193.6 mm
- net col8: track 153.0 -> 152.2 mm
- net col10: track 218.5 -> 217.7 mm
Other:
- outline, holes or cut-outs redrawn

Commit message: update pcb common and update goose45 key loaction
Parts:
- removed R6: 10K/5%, Resistor_SMD:R_0603_1608Metric
- added SW37_1: SW_Push, Switch_Keyboard_Hotswap_Kailh.pretty:SW_Hotswap_Kailh_MX, F.Cu at (242.5, 105.1)
- added SW38_1: SW_Push, Switch_Keyboard_Hotswap_Kailh.pretty:SW_Hotswap_Kailh_MX, F.Cu at (264.0, 105.1)
- moved D37 10.7 mm to (233.1, 111.8), turned to 90 degrees
- moved D38 7.14 mm to (257.1, 113.7)
- turned SW38 to 0 degrees
- turned SW37 to 0 degrees
Connections:
- SW28 pad 2: col2 -> col2_1
- SW40 pad 2: col2 -> col2_1
- SW40_1 pad 1: col2 -> col2_1
- U1 pad 12: PA2 -> col2_1
Routing:
- net col2: track 143.0 -> 32.6 mm, vias 4 -> 2
- net col2_1: track 0.00 -> 48.0 mm, vias 0 -> 2
- net PA2: track 28.5 -> 0.00 mm, vias 2 -> 0
- net col12: track 252.8 -> 268.0 mm, vias 2 -> 3
- net col11: track 240.8 -> 250.0 mm, vias 2 -> 3
- net row3: track 259.7 -> 253.5 mm, vias 12 -> 11
- net Net-(D38-Pad2): track 7.45 -> 12.6 mm
- net Net-(D37-Pad2): track 7.10 -> 12.0 mm
- net GND: track 393.8 -> 392.3 mm, vias 325 -> 321
- net row4: track 297.8 -> 298.4 mm, vias 6 -> 7
