File: goose45rev1/switchs.kicad_sch (KiCad schematic)
At the start: 90 parts, among them SW10 SW_Push, SW11 SW_Push, SW12 SW_Push, SW13 SW_Push, SW14 SW_Push, SW15 SW_Push, SW16 SW_Push, SW17 SW_Push, SW18 SW_Push, SW19 SW_Push, SW20 SW_Push, SW21 SW_Push, SW22 SW_Push, SW23 SW_Push, SW24 SW_Push, SW25 SW_Push, SW26 SW_Push, SW27 SW_Push, SW28 SW_Push, SW29 SW_Push, SW3 SW_Push, SW30 SW_Push, SW31 SW_Push, SW32 SW_Push, SW33 SW_Push, SW34 SW_Push, SW35 SW_Push, SW36 SW_Push, SW37 SW_Push, SW38 SW_Push, SW39 SW_Push, SW4 SW_Push, SW40 SW_Push, SW41 SW_Push, SW42 SW_Push, SW43 SW_Push, SW44 SW_Push, SW45 SW_Push, SW46 SW_Push, SW48 SW_Push, SW5 SW_Push, SW6 SW_Push, SW7 SW_Push, SW8 SW_Push, SW9 SW_Push

Commit message: change Diode pcb pad and modify usb connector location
Parts:
- D10, D11, D12, D13, D14, D15, D16, D17, D18, D19, D20, D21, D22, D23, D24, D25, D26, D27, D28, D29, D3, D30, D31, D32, D33, D34, D35, D36, D37, D38, D39, D4, D40, D41, D42, D43, D44, D45, D46, D48, D5, D6, D7, D8, D9: footprint Diode_SMD:D_0805_2012Metric -> Diode_SMD:D_SOD-323

Commit message: Change goose45 mod key size
Parts:
- added SW39_1, SW40_1, SW41_1, SW44_1: SW_Push, Switch_Keyboard_Hotswap_Kailh.pretty:SW_Hotswap_Kailh_MX, symbol Switch:SW_Push
Connections:
- net col1: now also SW39_1.2
- net col2: now also SW40_1.1
- net col3: now also SW41.2, SW41_1.1; no longer SW41.1
- net col9: now also SW44.1, SW44_1.2; no longer SW44.2
- net at D39.2 (A), SW39.2: now also SW39_1.1
- net at D41.2 (A): now also SW41.1, SW41_1.2; no longer SW41.2
- net at D44.2 (A): now also SW44.2, SW44_1.1; no longer SW44.1
- net at D40.2 (A), SW40.1: now also SW40_1.2
Other:
- moved on the sheet: SW41, SW44

Commit message: update pcb common and update goose45 key loaction
Parts:
- added SW37_1, SW38_1: SW_Push, Switch_Keyboard_Hotswap_Kailh.pretty:SW_Hotswap_Kailh_MX, symbol Switch:SW_Push
Connections:
- net col11: now also SW37_1.1
- net col12: now also SW38_1.1
- net col2: no longer SW28.2, SW40.2, SW40_1.1
- net at D37.2 (A), SW37.1: now also SW37_1.2
- net at D38.2 (A), SW38.1: now also SW38_1.2
- new net col2_1: SW28.2, SW40.2, SW40_1.1
Changed lines of the file:
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@@
   (junction (at 304.8 74.93) (diameter 0) (color 0 0 0 0)
   )
-  (junction (at 105.41 129.54) (diameter 0) (color 0 0 0 0)
+  (junction (at 358.14 167.64) (diameter 0) (color 0 0 0 0)
   )
   (junction (at 62.23 203.2) (diameter 0) (color 0 0 0 0)
@@
   (junction (at 85.09 201.93) (diameter 0) (color 0 0 0 0)
   )
+  (junction (at 332.74 167.64) (diameter 0) (color 0 0 0 0)
+  )
   (junction (at 228.6 151.13) (diameter 0) (color 0 0 0 0)
   )
@@
   (junction (at 359.41 208.28) (diameter 0) (color 0 0 0 0)
   )
+  (junction (at 320.04 167.64) (diameter 0) (color 0 0 0 0)
+  )
   (junction (at 334.01 167.64) (diameter 0) (color 0 0 0 0)
   )
@@
   (junction (at 156.21 167.64) (diameter 0) (color 0 0 0 0)
   )
+  (junction (at 105.41 167.64) (diameter 0) (color 0 0 0 0)
+  )
   (junction (at 181.61 167.64) (diameter 0) (color 0 0 0 0)
   )
@@
   (junction (at 130.81 208.28) (diameter 0) (color 0 0 0 0)
   )
-  (junction (at 105.41 167.64) (diameter 0) (color 0 0 0 0)
-  )
   (junction (at 80.01 91.44) (diameter 0) (color 0 0 0 0)
   )
@@
   (junction (at 130.81 129.54) (diameter 0) (color 0 0 0 0)
   )
+  (junction (at 345.44 167.64) (diameter 0) (color 0 0 0 0)
+  )
   (junction (at 80.01 132.08) (diameter 0) (color 0 0 0 0)
   )
@@
   (junction (at 105.41 212.09) (diameter 0) (color 0 0 0 0)
   )
+  (wire (pts (xy 105.41 147.32) (xy 105.41 167.64))
+    (stroke (width 0) (type default) (color 0 0 0 0))
+  )
   (wire (pts (xy 91.44 129.54) (xy 92.71 129.54))
     (stroke (width 0) (type default) (color 0 0 0 0))
@@
     (stroke (width 0) (type default) (color 0 0 0 0))
   )
+  (wire (pts (xy 356.87 171.45) (xy 358.14 171.45))
+    (stroke (width 0) (type default) (color 0 0 0 0))
+  )
   (wire (pts (xy 119.38 119.38) (xy 116.84 119.38))
     (stroke (width 0) (type default) (color 0 0 0 0))
@@
     (stroke (width 0) (type default) (color 0 0 0 0))
   )
+  (wire (pts (xy 346.71 171.45) (xy 345.44 171.45))
+    (stroke (width 0) (type default) (color 0 0 0 0))
+  )
   (wire (pts (xy 128.27 208.28) (xy 130.81 208.28))
     (stroke (width 0) (type default) (color 0 0 0 0))
   )
+  (wire (pts (xy 358.14 171.45) (xy 358.14 167.64))
+    (stroke (width 0) (type default) (color 0 0 0 0))
+  )
   (wire (pts (xy 161.29 201.93) (xy 163.83 201.93))
     (stroke (width 0) (type default) (color 0 0 0 0))
@@
     (stroke (width 0) (type default) (color 0 0 0 0))
   )
+  (wire (pts (xy 332.74 171.45) (xy 332.74 167.64))
+    (stroke (width 0) (type default) (color 0 0 0 0))
+  )
   (wire (pts (xy 177.8 151.13) (xy 203.2 151.13))
     (stroke (width 0) (type default) (color 0 0 0 0))
@@
     (stroke (width 0) (type default) (color 0 0 0 0))
   )
+  (wire (pts (xy 110.49 147.32) (xy 105.41 147.32))
+    (stroke (width 0) (type default) (color 0 0 0 0))
+  )
+  (wire (pts (xy 331.47 171.45) (xy 332.74 171.45))
+    (stroke (width 0) (type default) (color 0 0 0 0))
+  )
   (wire (pts (xy 177.8 113.03) (xy 177.8 119.38))
     (stroke (width 0) (type default) (color 0 0 0 0))
@@
     (stroke (width 0) (type default) (color 0 0 0 0))
   )
+  (wire (pts (xy 321.31 171.45) (xy 320.04 171.45))
+    (stroke (width 0) (type default) (color 0 0 0 0))
+  )
   (wire (pts (xy 179.07 167.64) (xy 181.61 167.64))
     (stroke (width 0) (type default) (color 0 0 0 0))
   )
+  (wire (pts (xy 110.49 59.69) (xy 110.49 147.32))
+    (stroke (width 0) (type default) (color 0 0 0 0))
+  )
   (wire (pts (xy 322.58 119.38) (xy 320.04 119.38))
     (stroke (width 0) (type default) (color 0 0 0 0))
@@
     (stroke (width 0) (type default) (color 0 0 0 0))
   )
+  (wire (pts (xy 320.04 171.45) (xy 320.04 167.64))
+    (stroke (width 0) (type default) (color 0 0 0 0))
+  )
   (wire (pts (xy 181.61 91.44) (xy 181.61 129.54))
     (stroke (width 0) (type default) (color 0 0 0 0))
@@
     (stroke (width 0) (type default) (color 0 0 0 0))
   )
-  (wire (pts (xy 105.41 129.54) (xy 105.41 167.64))
-    (stroke (width 0) (type default) (color 0 0 0 0))
-  )
   (wire (pts (xy 167.64 157.48) (xy 167.64 167.64))
     (stroke (width 0) (type default) (color 0 0 0 0))
@@
     (stroke (width 0) (type default) (color 0 0 0 0))
   )
+  (wire (pts (xy 358.14 167.64) (xy 359.41 167.64))
+    (stroke (width 0) (type default) (color 0 0 0 0))
+  )
   (wire (pts (xy 91.44 167.64) (xy 92.71 167.64))
     (stroke (width 0) (type default) (color 0 0 0 0))
@@
     (stroke (width 0) (type default) (color 0 0 0 0))
   )
+  (wire (pts (xy 345.44 171.45) (xy 345.44 167.64))
+    (stroke (width 0) (type default) (color 0 0 0 0))
+  )
   (wire (pts (xy 283.21 167.64) (xy 283.21 208.28))
     (stroke (width 0) (type default) (color 0 0 0 0))
@@
     (stroke (width 0) (type default) (color 0 0 0 0))
   )
-  (wire (pts (xy 331.47 167.64) (xy 334.01 167.64))
-    (stroke (width 0) (type default) (color 0 0 0 0))
-  )
-  (wire (pts (xy 356.87 167.64) (xy 359.41 167.64))
+  (wire (pts (xy 331.47 167.64) (xy 332.74 167.64))
+    (stroke (width 0) (type default) (color 0 0 0 0))
+  )
+  (wire (pts (xy 356.87 167.64) (xy 358.14 167.64))
+    (stroke (width 0) (type default) (color 0 0 0 0))
+  )
+  (wire (pts (xy 332.74 167.64) (xy 334.01 167.64))
     (stroke (width 0) (type default) (color 0 0 0 0))
   )
@@
     (effects (font (size 1.27 1.27)) (justify left))
   )
+  (hierarchical_label "col2_1" (shape bidirectional) (at 110.49 59.69 90)
+    (effects (font (size 1.27 1.27)) (justify left))
+  )
   (symbol (lib_id "Diode:1N4148") (at 299.72 195.58 180) (unit 1)
     (in_bom yes) (on_board yes)
@@
   (symbol (lib_id "Switch:SW_Push") (at 326.39 167.64 0) (unit 1)
     (in_bom yes) (on_board yes)
-    (property "Reference" "SW37" (id 0) (at 326.39 171.45 0))
+    (property "Reference" "SW37" (id 0) (at 323.85 163.83 0))
     (property "Value" "SW_Push" (id 1) (at 326.39 162.56 0)
       (effects (font (size 1.27 1.27)) hide)
@@
     (pin "2")
   )
+  (symbol (lib_id "Switch:SW_Push") (at 326.39 171.45 180) (unit 1)
+    (in_bom yes) (on_board yes)
+    (property "Reference" "SW37_1" (id 0) (at 320.04 173.99 0))
+    (property "Value" "SW_Push" (id 1) (at 326.39 176.53 0)
+      (effects (font (size 1.27 1.27)) hide)
+    )
+    (property "Footprint" "Switch_Keyboard_Hotswap_Kailh.pretty:SW_Hotswap_Kailh_MX" (id 2) (at 326.39 176.53 0)
+      (effects (font (size 1.27 1.27)) hide)
+    )
+    (property "Datasheet" "~" (id 3) (at 326.39 176.53 0)
+      (effects (font (size 1.27 1.27)) hide)
+    )
+    (pin "1")
+    (pin "2")
+  )
   (symbol (lib_id "Switch:SW_Push") (at 173.99 167.64 0) (unit 1)
     (in_bom yes) (on_board yes)
@@
     (pin "2")
   )
+  (symbol (lib_id "Switch:SW_Push") (at 351.79 171.45 180) (unit 1)
+    (in_bom yes) (on_board yes)
+    (property "Reference" "SW38_1" (id 0) (at 346.71 173.99 0))
+    (property "Value" "SW_Push" (id 1) (at 351.79 176.53 0)
+      (effects (font (size 1.27 1.27)) hide)
+    )
+    (property "Footprint" "Switch_Keyboard_Hotswap_Kailh.pretty:SW_Hotswap_Kailh_MX" (id 2) (at 351.79 176.53 0)
+      (effects (font (size 1.27 1.27)) hide)
+    )
+    (property "Datasheet" "~" (id 3) (at 351.79 176.53 0)
+      (effects (font (size 1.27 1.27)) hide)
+    )
+    (pin "1")
+    (pin "2")
+  )
   (symbol (lib_id "Switch:SW_Push") (at 148.59 91.44 0) (unit 1)
     (in_bom yes) (on_board yes)
@@
   (symbol (lib_id "Switch:SW_Push") (at 351.79 167.64 0) (unit 1)
     (in_bom yes) (on_board yes)
-    (property "Reference" "SW38" (id 0) (at 351.79 171.45 0))
+    (property "Reference" "SW38" (id 0) (at 349.25 163.83 0))
     (property "Value" "SW_Push" (id 1) (at 351.79 162.56 0)
       (effects (font (size 1.27 1.27)) hide)
