File: goose45rev1/power_manager.kicad_sch (KiCad schematic)
At the start: 11 parts, among them U3 TLV75533PDBV

Commit message: change Diode pcb pad and modify usb connector location
Parts:
- D2: footprint Diode_SMD:D_0805_2012Metric -> Diode_SMD:D_SOD-323
Changed lines of the file:
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@@
     (property "Reference" "D2" (id 0) (at 148.082 75.184 0))
     (property "Value" "1N4148" (id 1) (at 148.082 77.724 0))
-    (property "Footprint" "Diode_SMD:D_0805_2012Metric" (id 2) (at 148.082 85.725 0)
+    (property "Footprint" "Diode_SMD:D_SOD-323" (id 2) (at 148.082 85.725 0)
       (effects (font (size 1.27 1.27)) hide)
     )

Commit message: change goose45 power module foodpoint
Parts:
- C12, C13: footprint Capacitor_SMD:C_1206_3216Metric -> Capacitor_SMD:C_0603_1608Metric
Changed lines of the file:
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@@
       (effects (font (size 1.27 1.27)) (justify left))
     )
-    (property "Footprint" "Capacitor_SMD:C_1206_3216Metric" (id 2) (at 170.942 117.094 0)
+    (property "Footprint" "Capacitor_SMD:C_0603_1608Metric" (id 2) (at 170.942 117.094 0)
       (effects (font (size 1.27 1.27)) hide)
     )
@@
       (effects (font (size 1.27 1.27)) (justify left))
     )
-    (property "Footprint" "Capacitor_SMD:C_1206_3216Metric" (id 2) (at 97.536 117.094 0)
+    (property "Footprint" "Capacitor_SMD:C_0603_1608Metric" (id 2) (at 97.536 117.094 0)
       (effects (font (size 1.27 1.27)) hide)
     )
