File: usbhub2.0/usbhub2.0.kicad_pcb (KiCad board)
At the start: 2 copper layers, 73 x 38.3 mm, 28 parts, among them J1 Conn_01x05_Male, J2 Conn_01x05_Male, J3 Power, J4 Conn_01x05_Male, J5 USB_C_Receptacle_USB2.0, J7 Conn_01x05_Male, J9 Power, U1 FE1.1s, Y1 Crystal_12MHz

Commit message: modify the usbhub2.0 board edge
Routing:
- net GND: vias 81 -> 83
Other:
- board size 73 x 38.3 mm -> 79 x 38.3 mm

Commit message: update usbhub 2.0 board edge size and the comment
Other:
- board size 79 x 38.3 mm -> 81 x 38.3 mm
Changed lines of the file:
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@@
     )
   )
-  (gr_line (start 85.515 114.11) (end 89.015 114.11) (layer "Cmts.User") (width 0.15))
   (gr_line locked (start 99.48 79.31) (end 108.64 79.31) (layer "Edge.Cuts") (width 0.1))
   (gr_arc locked (start 108.64 79.31) (mid 108.993553 79.456447) (end 109.14 79.81) (layer "Edge.Cuts") (width 0.1))
   (gr_line locked (start 164.5 82.61) (end 164.5 117.61) (layer "Edge.Cuts") (width 0.1))
   (gr_line locked (start 109.14 82.61) (end 164.5 82.61) (layer "Edge.Cuts") (width 0.1))
-  (gr_circle (center 89.015 114.11) (end 90.615 114.11) (layer "Edge.Cuts") (width 0.1) (fill none))
-  (gr_line locked (start 85.515 117.61) (end 164.5 117.61) (layer "Edge.Cuts") (width 0.1))
+  (gr_circle (center 87.015 114.11) (end 88.615 114.11) (layer "Edge.Cuts") (width 0.1) (fill none))
+  (gr_line locked (start 83.515 117.61) (end 164.5 117.61) (layer "Edge.Cuts") (width 0.1))
   (gr_line locked (start 98.98 79.81) (end 98.98 82.61) (layer "Edge.Cuts") (width 0.1))
   (gr_circle (center 161 86.11) (end 162.6 86.11) (layer "Edge.Cuts") (width 0.1) (fill none))
@@
   (gr_arc (start 98.98 79.81) (mid 99.126447 79.456447) (end 99.48 79.31) (layer "Edge.Cuts") (width 0.1))
   (gr_circle (center 161 114.11) (end 162.6 114.11) (layer "Edge.Cuts") (width 0.1) (fill none))
-  (gr_line locked (start 85.515 82.61) (end 85.515 117.61) (layer "Edge.Cuts") (width 0.1))
-  (gr_circle (center 89.015 86.11) (end 90.615 86.11) (layer "Edge.Cuts") (width 0.1) (fill none))
-  (gr_line locked (start 85.515 82.61) (end 98.98 82.61) (layer "Edge.Cuts") (width 0.1))
+  (gr_line locked (start 83.515 82.61) (end 83.515 117.61) (layer "Edge.Cuts") (width 0.1))
+  (gr_circle (center 87.015 86.11) (end 88.615 86.11) (layer "Edge.Cuts") (width 0.1) (fill none))
+  (gr_line locked (start 83.515 82.61) (end 98.98 82.61) (layer "Edge.Cuts") (width 0.1))
   (gr_text "Design in Taiwan\n2022.12" (at 101.07 113.61) (layer "F.SilkS")
     (effects (font (size 0.5 0.5) (thickness 0.1)))
@@
   )
   (dimension (type aligned) (layer "Cmts.User")
-    (pts (xy 85.515 114.11) (xy 89.015 114.11))
-    (height 12.99)
-    (gr_text "3.5000 mm" (at 87.265 125.95) (layer "Cmts.User")
-      (effects (font (size 1 1) (thickness 0.15)) (justify left))
+    (pts (xy 87.015 86.11) (xy 104.06 86.11))
+    (height -11.36)
+    (gr_text "17.0450 mm" (at 95.5375 73.6) (layer "Cmts.User")
+      (effects (font (size 1 1) (thickness 0.15) italic) (justify right))
     )
     (format (units 3) (units_format 1) (precision 4))
@@
   )
   (dimension (type aligned) (layer "Cmts.User")
-    (pts (xy 89.015 114.11) (xy 161 114.11))
-    (height 18.939999)
-    (gr_text "71.9850 mm" (at 125.0075 131.899999) (layer "Cmts.User")
-      (effects (font (size 1 1) (thickness 0.15)))
-    )
-    (format (units 3) (units_format 1) (precision 4))
-    (style (thickness 0.15) (arrow_length 1.27) (text_position_mode 0) (extension_height 0.58642) (extension_offset 0.5) keep_text_aligned)
-  )
-  (dimension (type aligned) (layer "Cmts.User")
-    (pts (xy 89.015 115.71) (xy 89.015 112.51))
-    (height -12.665)
-    (gr_text "3.2000 mm" (at 75.2 114.11 90) (layer "Cmts.User")
-      (effects (font (size 1 1) (thickness 0.15)) (justify left))
+    (pts (xy 87.015 115.71) (xy 87.015 112.51))
+    (height -10.615)
+    (gr_text "3.2000 mm" (at 75.25 114.11 90) (layer "Cmts.User")
+      (effects (font (size 1 1) (thickness 0.15) italic) (justify left))
     )
     (format (units 3) (units_format 1) (precision 4))
@@
   )
   (dimension (type aligned) (layer "Cmts.User")
-    (pts (xy 89.015 114.11) (xy 89.015 117.61))
-    (height 17.265)
-    (gr_text "3.5000 mm" (at 70.6 115.86 90) (layer "Cmts.User")
-      (effects (font (size 1 1) (thickness 0.15)) (justify left))
+    (pts (xy 83.515 82.61) (xy 98.98 82.61))
+    (height -14.66)
+    (gr_text "15.4650 mm" (at 91.2475 66.8) (layer "Cmts.User")
+      (effects (font (size 1 1) (thickness 0.15) italic) (justify left))
     )
     (format (units 3) (units_format 1) (precision 4))
@@
     (height -24.28)
     (gr_text "3.3000 mm" (at 73.55 80.96 90) (layer "Cmts.User")
-      (effects (font (size 1 1) (thickness 0.15)) (justify left))
+      (effects (font (size 1 1) (thickness 0.15) italic) (justify left))
     )
     (format (units 3) (units_format 1) (precision 4))
@@
   )
   (dimension (type aligned) (layer "Cmts.User")
-    (pts (xy 85.515 82.61) (xy 98.98 82.61))
-    (height -14.71)
-    (gr_text "13.4650 mm" (at 92.2475 66.75) (layer "Cmts.User")
-      (effects (font (size 1 1) (thickness 0.15)) (justify left))
+    (pts (xy 87.015 114.11) (xy 87.015 117.61))
+    (height 15.365)
+    (gr_text "3.5000 mm" (at 70.5 115.86 90) (layer "Cmts.User")
+      (effects (font (size 1 1) (thickness 0.15) italic) (justify left))
+    )
+    (format (units 3) (units_format 1) (precision 4))
+    (style (thickness 0.15) (arrow_length 1.27) (text_position_mode 0) (extension_height 0.58642) (extension_offset 0.5) keep_text_aligned)
+  )
+  (dimension (type aligned) (layer "Cmts.User")
+    (pts (xy 87.015 114.11) (xy 161 114.11))
+    (height 13.739999)
+    (gr_text "73.9850 mm" (at 124.0075 126.699999) (layer "Cmts.User")
+      (effects (font (size 1 1) (thickness 0.15) italic))
     )
     (format (units 3) (units_format 1) (precision 4))
@@
   )
   (dimension (type aligned) (layer "Cmts.User")
-    (pts (xy 89.015 86.11) (xy 104.06 86.11))
-    (height -11.36)
-    (gr_text "15.0450 mm" (at 96.5375 73.6) (layer "Cmts.User")
-      (effects (font (size 1 1) (thickness 0.15)))
+    (pts (xy 83.515 82.61) (xy 164.5 82.61))
+    (height -22.76)
+    (gr_text "80.9850 mm" (at 124.0075 58.7) (layer "Cmts.User")
+      (effects (font (size 1 1) (thickness 0.15) italic))
     )
     (format (units 3) (units_format 1) (precision 4))
-    (style (thickness 0.15) (arrow_length 1.27) (text_position_mode 0) (extension_height 0.58642) (extension_offset 0.5) keep_text_aligned)
-  )
-  (dimension (type aligned) (layer "Cmts.User")
-    (pts (xy 85.515 82.61) (xy 164.5 82.61))
-    (height -22.86)
-    (gr_text "78.9850 mm" (at 125.0075 58.6) (layer "Cmts.User")
-      (effects (font (size 1 1) (thickness 0.15)))
-    )
-    (format (units 3) (units_format 1) (precision 4))
