File: usbhub2.0rev2/usbhub2.0rev2.kicad_pcb (KiCad board)
At the start: 2 copper layers, 100 x 40.6 mm, 25 parts, among them J1 Conn_01x12_Pin, J10 Power, J2 Conn_01x05_Male, J3 Conn_01x12_Pin, J4 USB_C_Receptacle_USB2.0, J9 Power, U1 FE1.1s, Y1 Crystal_12MHz

Commit message: add goose45 rev3 and usbhub2.3 rev2
Routing:
- net GND: track 246.2 -> 246.3 mm, vias 56 -> 57
Other:
- board size 100 x 40.6 mm -> 100 x 35.1 mm
- board text added: "KiCAD shift X: 100mm Y: 50mm"
