File: usbhub2.0rev2/usbhub2.0.kicad_pcb (KiCad board)
At the start: 2 copper layers, 100 x 35.1 mm, 25 parts, among them J1 Conn_01x12_Pin, J10 Power, J2 Conn_01x05_Male, J3 Conn_01x12_Pin, J4 USB_C_Receptacle_USB2.0, J9 Power, U1 FE1.1s, Y1 Crystal_12MHz

Commit message: add goose45 case v10 and update sub-usb pcb
Parts:
- moved J3 15.8 mm to (162.0, 77.1)
- moved C15 15.2 mm to (156.3, 70.6)
- moved C8 14.7 mm to (152.0, 72.3)
- moved J1 13.8 mm to (164.0, 63.0)
- moved C14 13.2 mm to (158.3, 59.1)
- moved C7 12.4 mm to (154.6, 61.1)
- moved C13 8.47 mm to (134.2, 54.8), turned to 180 degrees
- moved J10 5.71 mm to (141.2, 52.1)
- moved J2 5.71 mm to (151.3, 58.6)
- moved C6 2.66 mm to (135.9, 58.4), turned to 180 degrees
Routing:
- net VIN: track 151.9 -> 126.8 mm, vias 5 -> 4
- net USB4_D-: track 49.7 -> 33.9 mm
- net USB3_D-: track 49.0 -> 33.2 mm
- net USB4_D+: track 49.7 -> 33.9 mm
- net USB3_D+: track 49.0 -> 33.2 mm
- net GND: track 246.3 -> 231.0 mm, vias 57 -> 43
- net USB2_D-: track 46.7 -> 33.0 mm
- net USB2_D+: track 46.7 -> 33.0 mm
- net USB1_D-: track 28.7 -> 23.7 mm
- net USB1_D+: track 28.0 -> 22.9 mm
Other:
- board size 100 x 35.1 mm -> 72.5 x 35.1 mm
- board text added: "2023.12 Design in Taiwan"
- board text added: "usbhub2.0 rev2"
